File: AWTD-001.kicad_pcb (KiCad board)
At the start: 2 copper layers, 37 parts, among them J1 ADXL345 module, J10 Adapter_Det2, J11 Neopixel1, J12 AS5600_R, J13 AS5600_L, J14 TCS34725, J15 Stepper_R, J16 Stepper_L, J17 VL53L1X_Front, J19 Conn_01x24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

Commit message: commit
Parts:
- moved C2 14.2 mm to (163.0, 103.0)
- moved U4 14.2 mm to (166.5, 112.0)
Changed lines of the file:
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@@
 	(footprint "Package_TO_SOT_THT:TO-220-3_Vertical"
 		(layer "F.Cu")
-		(at 155.54 121.05 180)
+		(at 166.54 112.05 180)
 		(descr "TO-220-3, Vertical, RM 2.54mm, see https://www.vishay.com/docs/66542/to-220-1.pdf, generated with kicad-footprint-generator TO_SOT_THT_generate.py")
 		(tags "TO-220-3 Vertical RM 2.54mm")
@@
 	(footprint "Capacitor_THT:C_Radial_D5.0mm_H5.0mm_P2.00mm"
 		(layer "F.Cu")
-		(at 152 112)
+		(at 163 103)
 		(descr "C, Radial series, Radial, pin pitch=2.00mm, diameter=5mm, height=5mm, Non-Polar Electrolytic Capacitor")
 		(tags "C Radial series Radial pin pitch 2.00mm diameter 5mm height 5mm Non-Polar Electrolytic Capacitor")
